File: Arduino_Pro_Mini_PTH.sch (KiCad schematic (older format))
At the start: 24 parts, among them IC1 ATMEGA328P-PU, P1 I/O lo, P2 FTDI Basic, P3 A4 A5, P4 I/O hi, SW1 Reset, U1 L4931CZ50-AP, X1 8/16MHz

Commit message: Schematic complete.
Parts:
- removed C5, C6: TBD, ~, symbol C
- removed X1: 8/16MHz, ~, symbol CRYSTAL
- added X?: CSTLS16M0X53-B0, ~, symbol CRYSTAL_SMD
- D1, D2: footprint ~ -> LED-3MM
- JP1: value low_pwr -> LP
Connections:
- wire segments 198 -> 195
Other:
- note added: "6mm N.O. tactile\n(e.g. TE 1977120-6,\nC&K PTS645SL43 LFS)"
Changed lines of the file:
@@
 Sheet 1 1
 Title "Arduino Pro Mini using through-hole parts"
-Date "25 mar 2015"
+Date "26 mar 2015"
 Rev ""
 Comp "Mithat Konar (https://github.com/mithat/Arduino_Pro_Mini_PTH)"
-Comment1 "Pro Mini design by SparkFun Electronics (github.com/sparkfun/Arduino_Pro_Mini_328)"
+Comment1 "Original Pro Mini design by SparkFun Electronics"
 Comment2 "Creative Commons Attribution Share Alike 3.0 License"
 Comment3 ""
@@
 $EndComp
 $Comp
-L CRYSTAL X1
-U 1 1 55121E8C
-P 5600 4050
-F 0 "X1" H 5600 4200 60  0000 C CNN
-F 1 "8/16MHz" H 5600 3900 60  0000 C CNN
-F 2 "~" H 5600 4050 60  0000 C CNN
-F 3 "~" H 5600 4050 60  0000 C CNN
-	1    5600 4050
-	0    -1   -1   0
-$EndComp
-$Comp
-L C C5
-U 1 1 55121E9B
-P 5350 3700
-F 0 "C5" H 5350 3800 40  0000 L CNN
-F 1 "TBD" H 5356 3615 40  0000 L CNN
-F 2 "~" H 5388 3550 30  0000 C CNN
-F 3 "~" H 5350 3700 60  0000 C CNN
-	1    5350 3700
-	0    -1   -1   0
-$EndComp
-$Comp
-L C C6
-U 1 1 55121EA8
-P 5350 4400
-F 0 "C6" H 5350 4500 40  0000 L CNN
-F 1 "TBD" H 5356 4315 40  0000 L CNN
-F 2 "~" H 5388 4250 30  0000 C CNN
-F 3 "~" H 5350 4400 60  0000 C CNN
-	1    5350 4400
-	0    -1   -1   0
-$EndComp
-$Comp
 L GND #PWR01
 U 1 1 55121F28
-P 5000 4100
-F 0 "#PWR01" H 5000 4100 30  0001 C CNN
-F 1 "GND" H 5000 4030 30  0001 C CNN
-F 2 "" H 5000 4100 60  0000 C CNN
-F 3 "" H 5000 4100 60  0000 C CNN
-	1    5000 4100
+P 5350 4200
+F 0 "#PWR01" H 5350 4200 30  0001 C CNN
+F 1 "GND" H 5350 4130 30  0001 C CNN
+F 2 "" H 5350 4200 60  0000 C CNN
+F 3 "" H 5350 4200 60  0000 C CNN
+	1    5350 4200
 	1    0    0    -1
 $EndComp
@@
 F 0 "D2" H 8350 3150 50  0000 C CNN
 F 1 "LED" H 8350 2950 50  0000 C CNN
-F 2 "~" H 8350 3050 60  0000 C CNN
+F 2 "LED-3MM" H 8350 3050 60  0001 C CNN
 F 3 "~" H 8350 3050 60  0000 C CNN
 	1    8350 3050
@@
 	1    0    0    -1
 $EndComp
-Text Notes 8550 3100 1    60   ~ 0
+Text Notes 8550 3100 1    40   ~ 0
 Green
 $Comp
@@
 A4
 Wire Wire Line
-	5550 3700 5850 3700
-Wire Wire Line
-	5600 3750 5600 3700
-Connection ~ 5600 3700
-Wire Wire Line
 	5550 4400 5850 4400
 Wire Wire Line
-	5600 4350 5600 4400
-Connection ~ 5600 4400
-Wire Wire Line
-	5150 3700 5100 3700
-Wire Wire Line
-	5100 3700 5100 4400
-Wire Wire Line
-	5100 4400 5150 4400
-Wire Wire Line
-	5100 4050 5000 4050
-Wire Wire Line
-	5000 4050 5000 4100
-Connection ~ 5100 4050
+	5450 4150 5350 4150
+Wire Wire Line
+	5350 4150 5350 4200
 Wire Wire Line
 	6100 4850 6100 4750
@@
 Wire Wire Line
 	6150 4150 5850 4150
-Wire Wire Line
-	5850 4150 5850 3700
 Wire Wire Line
 	4750 2850 4750 2950
@@
 63 98 05 E1 6B C4 72 91 8E EA 95 27 8C 4B 0B 6B 30 6B 95 2D 08 DF 47 79 14 D8 40 20 A9 90 96 2D
 E1 E7 3D C6 74 F3 E0 6E B9 00 E4 0E CC EC 2A 00 9E 03 F9 2E 43 53 93 3B E7 B1 3D FE 0F E4 2C B5
-B8 3A B8 3B 5D 00 00 00 00 49 45 4E 44 AE 42 60 82 CB $EndBitmap
+B8 3A B8 3B 5D 00 00 00 00 49 45 4E 44 AE 42 60 82 65 $EndBitmap
 EndData
 $EndBitmap
@@
 F 0 "D1" H 2900 1650 50  0000 C CNN
 F 1 "LED" H 2900 1450 50  0000 C CNN
-F 2 "~" H 2900 1550 60  0000 C CNN
+F 2 "LED-3MM" H 2900 1550 60  0001 C CNN
 F 3 "~" H 2900 1550 60  0000 C CNN
 	1    2900 1550
@@
 	1    0    0    -1
 $EndComp
-Text Notes 3100 1650 1    60   ~ 0
+Text Notes 3100 1600 1    40   ~ 0
 Red
 $Comp
@@
 P 3350 1250
 F 0 "JP1" H 3350 1400 60  0000 C CNN
-F 1 "low_pwr" H 3350 1170 40  0000 C CNN
+F 1 "LP" H 3350 1170 40  0000 C CNN
 F 2 "~" H 3350 1250 60  0000 C CNN
 F 3 "~" H 3350 1250 60  0000 C CNN
@@
 Wire Wire Line
 	2900 2450 2900 2350
+Text Notes 3900 3900 0    40   ~ 0
+6mm N.O. tactile\n(e.g. TE 1977120-6,\nC&K PTS645SL43 LFS)
+$Comp
+L CRYSTAL_SMD X?
+U 1 1 55136729
+P 5550 4150
+F 0 "X?" H 5550 4240 40  0000 C CNN
+F 1 "CSTLS16M0X53-B0" H 5550 4300 30  0000 C CNN
+F 2 "~" H 5550 4150 60  0000 C CNN
+F 3 "~" H 5550 4150 60  0000 C CNN
+	1    5550 4150
+	0    1    1    0
+$EndComp
+Wire Wire Line
+	5550 4400 5550 4350
+Wire Wire Line
+	5550 3950 5550 3900
+Wire Wire Line
+	5550 3900 5850 3900
+Wire Wire Line
+	5850 3900 5850 4150
 $EndSCHEMATC

Commit message: Module associations.
Parts:
- C1, C2: footprint ~ -> mfk-CRP_5.0_2.0_0.5
- C3, C4, C7, C8: footprint ~ -> mfk-C_4.0_2.5_2.5_0.5
- IC1: footprint DIL28 -> mfk-DIP-28_300_rnd
- JP1: footprint ~ -> mfk-SIL-2
- P1, P4: footprint (none) -> mfk-SIL-12
- P2: footprint (none) -> mfk-SIL-6
- P3: footprint (none) -> mfk-SIL-2
- R1, R2, R3, R4, R5: footprint ~ -> mfk-R_0.25W_RN55_vert
- SW1: footprint ~ -> mfk-SW_PUSH_6MM
- U1: footprint TO-92-321 -> mfk-TO-92_f321
- X1: renamed from X?; footprint ~ -> mfk-Murata-CSTLS_X
Changed lines of the file:
@@
 F 0 "IC1" H 6300 5900 40  0000 L BNN
 F 1 "ATMEGA328P-PU" H 7400 3250 40  0000 L BNN
-F 2 "DIL28" H 7050 4650 30  0000 C CIN
+F 2 "mfk-DIP-28_300_rnd" H 7050 4650 30  0001 C CIN
 F 3 "~" H 7050 4650 60  0000 C CNN
 	1    7100 4650
@@
 F 0 "C7" H 5750 4900 40  0000 L CNN
 F 1 "100n" H 5756 4715 40  0000 L CNN
-F 2 "~" H 5788 4650 30  0000 C CNN
+F 2 "mfk-C_4.0_2.5_2.5_0.5" H 5788 4650 30  0001 C CNN
 F 3 "~" H 5750 4800 60  0000 C CNN
 	1    5750 4800
@@
 F 0 "C8" H 5750 5600 40  0000 L CNN
 F 1 "100n" H 5756 5415 40  0000 L CNN
-F 2 "~" H 5788 5350 30  0000 C CNN
+F 2 "mfk-C_4.0_2.5_2.5_0.5" H 5788 5350 30  0001 C CNN
 F 3 "~" H 5750 5500 60  0000 C CNN
 	1    5750 5500
@@
 F 0 "R2" V 4830 3200 40  0000 C CNN
 F 1 "10K" V 4757 3201 40  0000 C CNN
-F 2 "~" V 4680 3200 30  0000 C CNN
+F 2 "mfk-R_0.25W_RN55_vert" V 4680 3200 30  0001 C CNN
 F 3 "~" H 4750 3200 30  0000 C CNN
 	1    4750 3200
@@
 F 0 "SW1" H 4900 4060 50  0000 C CNN
 F 1 "Reset" H 4750 3870 50  0000 C CNN
-F 2 "~" H 4750 3950 60  0000 C CNN
+F 2 "mfk-SW_PUSH_6MM" H 4750 3950 60  0001 C CNN
 F 3 "~" H 4750 3950 60  0000 C CNN
 	1    4750 3950
@@
 F 0 "C4" H 4350 3650 40  0000 L CNN
 F 1 "100n" H 4356 3465 40  0000 L CNN
-F 2 "~" H 4388 3400 30  0000 C CNN
+F 2 "mfk-C_4.0_2.5_2.5_0.5" H 4388 3400 30  0001 C CNN
 F 3 "~" H 4350 3550 60  0000 C CNN
 	1    4350 3550
@@
 F 0 "P1" V 800 6050 60  0000 C CNN
 F 1 "I/O lo" V 900 6050 60  0000 C CNN
-F 2 "" H 850 6050 60  0000 C CNN
+F 2 "mfk-SIL-12" H 850 6050 60  0001 C CNN
 F 3 "" H 850 6050 60  0000 C CNN
 	1    850  6050
@@
 F 0 "P2" V 1900 3950 60  0000 C CNN
 F 1 "FTDI Basic" V 2000 3950 60  0000 C CNN
-F 2 "" H 1950 3950 60  0000 C CNN
+F 2 "mfk-SIL-6" H 1950 3950 60  0001 C CNN
 F 3 "" H 1950 3950 60  0000 C CNN
 	1    1950 3950
@@
 F 0 "P3" V 2300 7750 40  0000 C CNN
 F 1 "A4 A5" V 2400 7750 40  0000 C CNN
-F 2 "" H 2350 7750 60  0000 C CNN
+F 2 "mfk-SIL-2" H 2350 7750 60  0001 C CNN
 F 3 "" H 2350 7750 60  0000 C CNN
 	1    2350 7750
@@
 F 0 "P4" V 3300 6050 60  0000 C CNN
 F 1 "I/O hi" V 3400 6050 60  0000 C CNN
-F 2 "" H 3350 6050 60  0000 C CNN
+F 2 "mfk-SIL-12" H 3350 6050 60  0001 C CNN
 F 3 "" H 3350 6050 60  0000 C CNN
 	1    3350 6050
@@
 F 0 "R3" V 8430 2550 40  0000 C CNN
 F 1 "330" V 8357 2551 40  0000 C CNN
-F 2 "~" V 8280 2550 30  0000 C CNN
+F 2 "mfk-R_0.25W_RN55_vert" V 8280 2550 30  0001 C CNN
 F 3 "~" H 8350 2550 30  0000 C CNN
 	1    8350 2550
@@
 F 0 "R5" V 9980 3950 40  0000 C CNN
 F 1 "opt" V 9907 3951 40  0000 C CNN
-F 2 "~" V 9830 3950 30  0000 C CNN
+F 2 "mfk-R_0.25W_RN55_vert" V 9830 3950 30  0001 C CNN
 F 3 "~" H 9900 3950 30  0000 C CNN
 	1    9900 3950
@@
 F 0 "R4" V 9780 3950 40  0000 C CNN
 F 1 "opt" V 9707 3951 40  0000 C CNN
-F 2 "~" V 9630 3950 30  0000 C CNN
+F 2 "mfk-R_0.25W_RN55_vert" V 9630 3950 30  0001 C CNN
 F 3 "~" H 9700 3950 30  0000 C CNN
 	1    9700 3950
@@
 63 98 05 E1 6B C4 72 91 8E EA 95 27 8C 4B 0B 6B 30 6B 95 2D 08 DF 47 79 14 D8 40 20 A9 90 96 2D
 E1 E7 3D C6 74 F3 E0 6E B9 00 E4 0E CC EC 2A 00 9E 03 F9 2E 43 53 93 3B E7 B1 3D FE 0F E4 2C B5
-B8 3A B8 3B 5D 00 00 00 00 49 45 4E 44 AE 42 60 82 65 $EndBitmap
+B8 3A B8 3B 5D 00 00 00 00 49 45 4E 44 AE 42 60 82 9F $EndBitmap
 EndData
 $EndBitmap
@@
 F 0 "C1" H 1250 1650 50  0000 L CNN
 F 1 "10u" H 1250 1450 50  0000 L CNN
-F 2 "~" H 1200 1550 60  0000 C CNN
+F 2 "mfk-CRP_5.0_2.0_0.5" H 1200 1550 60  0001 C CNN
 F 3 "~" H 1200 1550 60  0000 C CNN
 	1    1200 1550
@@
 F 0 "R1" V 2980 2100 40  0000 C CNN
 F 1 "10K" V 2907 2101 40  0000 C CNN
-F 2 "~" V 2830 2100 30  0000 C CNN
+F 2 "mfk-R_0.25W_RN55_vert" V 2830 2100 30  0001 C CNN
 F 3 "~" H 2900 2100 30  0000 C CNN
 	1    2900 2100
@@
 F 0 "C2" H 3850 1700 50  0000 L CNN
 F 1 "10u" H 3850 1500 50  0000 L CNN
-F 2 "~" H 3800 1600 60  0000 C CNN
+F 2 "mfk-CRP_5.0_2.0_0.5" H 3800 1600 60  0001 C CNN
 F 3 "~" H 3800 1600 60  0000 C CNN
 	1    3800 1600
@@
 F 0 "C3" H 4150 1700 40  0000 L CNN
 F 1 "100n" H 4156 1515 40  0000 L CNN
-F 2 "~" H 4188 1450 30  0000 C CNN
+F 2 "mfk-C_4.0_2.5_2.5_0.5" H 4188 1450 30  0001 C CNN
 F 3 "~" H 4150 1600 60  0000 C CNN
 	1    4150 1600
@@
 F 0 "JP1" H 3350 1400 60  0000 C CNN
 F 1 "LP" H 3350 1170 40  0000 C CNN
-F 2 "~" H 3350 1250 60  0000 C CNN
+F 2 "mfk-SIL-2" H 3350 1250 60  0001 C CNN
 F 3 "~" H 3350 1250 60  0000 C CNN
 	1    3350 1250
@@
 F 0 "U1" H 1800 1500 40  0000 C CNN
 F 1 "L4931CZ50-AP" H 2000 1500 40  0000 L CNN
-F 2 "TO-92-321" H 2000 1400 30  0000 C CIN
+F 2 "mfk-TO-92_f321" H 2000 1400 30  0001 C CIN
 F 3 "~" H 2000 1300 60  0000 C CNN
 	1    2000 1300
@@
 6mm N.O. tactile\n(e.g. TE 1977120-6,\nC&K PTS645SL43 LFS)
 $Comp
-L CRYSTAL_SMD X?
+L CRYSTAL_SMD X1
 U 1 1 55136729
 P 5550 4150
-F 0 "X?" H 5550 4240 40  0000 C CNN
+F 0 "X1" H 5550 4240 40  0000 C CNN
 F 1 "CSTLS16M0X53-B0" H 5550 4300 30  0000 C CNN
-F 2 "~" H 5550 4150 60  0000 C CNN
+F 2 "mfk-Murata-CSTLS_X" H 5550 4150 60  0001 C CNN
 F 3 "~" H 5550 4150 60  0000 C CNN
 	1    5550 4150

Commit message: Routed.
Parts:
- removed JP1: LP, mfk-SIL-2, symbol JUMPER
Connections:
- net VCC: now also D1.1 (A), U1.3 (OUT)
Other:
- note added: "For low power application,\ndo not populate U1, D1, R1."
- note removed: "Power isolation jumper\n(for low power applications)"
Changed lines of the file:
@@
 63 98 05 E1 6B C4 72 91 8E EA 95 27 8C 4B 0B 6B 30 6B 95 2D 08 DF 47 79 14 D8 40 20 A9 90 96 2D
 E1 E7 3D C6 74 F3 E0 6E B9 00 E4 0E CC EC 2A 00 9E 03 F9 2E 43 53 93 3B E7 B1 3D FE 0F E4 2C B5
-B8 3A B8 3B 5D 00 00 00 00 49 45 4E 44 AE 42 60 82 9F $EndBitmap
+B8 3A B8 3B 5D 00 00 00 00 49 45 4E 44 AE 42 60 82 B5 $EndBitmap
 EndData
 $EndBitmap
@@
 Wire Wire Line
 	3800 1900 3800 1800
-$Comp
-L JUMPER JP1
-U 1 1 55123E65
-P 3350 1250
-F 0 "JP1" H 3350 1400 60  0000 C CNN
-F 1 "LP" H 3350 1170 40  0000 C CNN
-F 2 "mfk-SIL-2" H 3350 1250 60  0001 C CNN
-F 3 "~" H 3350 1250 60  0000 C CNN
-	1    3350 1250
-	1    0    0    -1
-$EndComp
 Wire Wire Line
 	2900 1350 2900 1250
 Wire Wire Line
-	2400 1250 3050 1250
-Wire Wire Line
-	4150 1250 3650 1250
+	2400 1250 4150 1250
 Wire Wire Line
 	4150 1100 4150 1400
@@
 $Comp
 L PWR_FLAG #FLG022
-U 1 1 551241A8
-P 4500 1150
-F 0 "#FLG022" H 4500 1245 30  0001 C CNN
-F 1 "PWR_FLAG" H 4500 1330 30  0000 C CNN
-F 2 "" H 4500 1150 60  0000 C CNN
-F 3 "" H 4500 1150 60  0000 C CNN
-	1    4500 1150
-	1    0    0    -1
-$EndComp
-Connection ~ 4150 1150
-Wire Wire Line
-	4500 1150 4150 1150
-$Comp
-L PWR_FLAG #FLG023
 U 1 1 5512446B
 P 4500 1800
-F 0 "#FLG023" H 4500 1895 30  0001 C CNN
+F 0 "#FLG022" H 4500 1895 30  0001 C CNN
 F 1 "PWR_FLAG" H 4500 1980 30  0000 C CNN
 F 2 "" H 4500 1800 60  0000 C CNN
@@
 	4500 1850 4500 1800
 Connection ~ 4150 1850
-Text Notes 3000 950  0    40   ~ 0
-Power isolation jumper\n(for low power applications)
 Text Notes 1800 1000 0    40   ~ 0
 20V max input
@@
 Connection ~ 2900 1250
 $Comp
-L GND #PWR024
+L GND #PWR023
 U 1 1 5512C102
 P 2000 1650
-F 0 "#PWR024" H 2000 1650 30  0001 C CNN
+F 0 "#PWR023" H 2000 1650 30  0001 C CNN
 F 1 "GND" H 2000 1580 30  0001 C CNN
 F 2 "" H 2000 1650 60  0000 C CNN
@@
 Wire Wire Line
 	5850 3900 5850 4150
+Text Notes 1700 1850 0    40   ~ 0
+For low power application,\ndo not populate U1, D1, R1.
 $EndSCHEMATC
